File: Electrical/PCB/MultiTB/MultiTB.sch (EAGLE design)
At the start: 9 parts, among them U2 TB6612FNG

Commit message: PCB Batch #1
Parts:
- added C11, C12: 0.1uF, Scott-Electrical:CAP_CERAMIC_0603
- added C13, C6: 10uF, Scott-Electrical:CAP_CERAMIC_0805
- added F1: 7A, Scott-Electrical:FUSE-1206
- added F2: 2A, Scott-Electrical:FUSE-0603
- added J1: (no value), SparkFun-Connectors:CONN_05
- added MACTRL, MBCTRL, MCCTRL, MDCTRL: JST_1.25_3P, Scott-Connectors:JST_1.25_3P
- added MC, MD: JST_XH_2.54_2P, Scott-Connectors:JST_XH_2.54_2P
- added MCU: JST_1.25_4P, Scott-Connectors:JST_1.25_4P
- added MCUC, MCUD: JST_1.25_5P, Scott-Connectors:JST_1.25_5P
- added R6: 10K, Scott-Electrical:RESISTOR0603
- added R8, R9: 10K, microbuilder:RESISTOR_4PACK
- added RPWM, RPWM2: 330, Scott-Electrical:RESISTOR_ARRAY_1206_SEPARATE_REVERSE
- added SJ_A12, SJ_A13, SJ_A14, SJ_A15, SJ_A16, SJ_A17: (no value), microbuilder:SOLDERJUMPERREFLOW_NOPASTE
- added TP13, TP14, TP15, TP16, TP17, TP18: (no value), microbuilder:TESTPOINTROUND2MM
- added U4: PCA9685, microbuilder:PCA9685
- added U5: TB6612FNG, SparkFun-IC-Special-Function:TB6612FNG
Connections:
- removed net STBY: U2.STBY
- removed net VCC: C2.1, MCUA.5, MCUB.5, U2.VCC
- new net 3.3V: C12.1, C2.1, C6.1, F2.1, MCUA.5, MCUB.5, MCUC.5, MCUD.5, SJ_A12.1, SJ_A13.1, SJ_A14.1, SJ_A15.1, SJ_A16.1, SJ_A17.1, U2.STBY, U2.VCC, U4.VDD, U5.STBY, U5.VCC
- new net A0: R9G$2.2, SJ_A12.2, TP13.P$1, U4.A0
- new net A1: R9G$1.2, SJ_A13.2, TP14.P$1, U4.A1
- new net A2: R8G$4.2, SJ_A14.2, TP15.P$1, U4.A2
- new net A3: R8G$3.2, SJ_A15.2, TP16.P$1, U4.A3
- new net A4: R8G$2.2, SJ_A16.2, TP17.P$1, U4.A4
- new net A5: R8G$1.2, SJ_A17.2, TP18.P$1, U4.A5
- new net C01: MC.1, U5.A01@1, U5.A01@2
- new net C02: MC.2, U5.A02@5, U5.A02@6
- new net CIN1: MCCTRL.1, MCUC.2, U5.AIN1
- new net CIN2: MCCTRL.3, MCUC.1, U5.AIN2
- new net D01: MD.1, U5.B01@11, U5.B01@12
- new net D02: MD.2, U5.B02@7, U5.B02@8
- new net DIN1: MCUD.2, MDCTRL.1, U5.BIN1
- new net DIN2: MCUD.1, MDCTRL.3, U5.BIN2
- new net N$1: J1.1, RPWM2@1.2
- new net N$2: F2.2, MCU.4
- new net N$3: J1.2, RPWM2@2.2
- new net N$4: J1.3, RPWM2@3.2
- new net N$5: J1.4, RPWM2@4.2
- new net OE: R6.1, U4.#OE
- new net PWM0: RPWM@1.1, U4.PWM0
- new net PWM1: RPWM@2.1, U4.PWM1
- new net PWM10: RPWM2@3.1, U4.PWM10
- new net PWM11: RPWM2@4.1, U4.PWM11
- new net PWM12: U4.PWM12
- new net PWM13: U4.PWM13
- new net PWM14: U4.PWM14
- new net PWM15: U4.PWM15
- new net PWM2: RPWM@3.1, U4.PWM2
- new net PWM3: RPWM@4.1, U4.PWM3
- new net PWM4: U4.PWM4
- new net PWM5: U4.PWM5
- new net PWM6: U4.PWM6
- new net PWM7: U4.PWM7
- new net PWM8: RPWM2@1.1, U4.PWM8
- new net PWM9: RPWM2@2.1, U4.PWM9
- new net PWMC: MCUC.3, RPWM@3.2, U5.PWMA
- new net PWMD: MCUD.3, RPWM@4.2, U5.PWMB
- new net SCL: MCU.1, U4.SCL
- new net SDA: MCU.2, U4.SDA
- new net VMIN: F1.1, PWR.1
- net AIN1: now also MACTRL.1
- net AIN2: now also MACTRL.3
- net BIN1: now also MBCTRL.1
- net BIN2: now also MBCTRL.3
- net GND: now also C11.2, C12.2, C13.2, C6.2, J1.5, MACTRL.2, MBCTRL.2, MCCTRL.2, MCU.3, MCUC.4, MCUD.4, MDCTRL.2, R6.2, R8G$1.1, R8G$2.1, R8G$3.1, R8G$4.1, R9G$1.1, R9G$2.1, U4.EXTCLK, U4.GND, U5.GND, U5.PGND1@3, U5.PGND1@4, U5.PGND2@10, U5.PGND2@9
- net PWMA: now also RPWM@1.2
- net PWMB: now also RPWM@2.2
- net VM: now also C11.1, C13.1, F1.2, U5.VM1, U5.VM2, U5.VM3; no longer PWR.1
