File: Electrical/PCB/TeensyBreakout/TeensyBreakout.brd (EAGLE design)
At the start: 29 x 47.2 mm, 7 parts, among them J1 TERMINAL

Commit message: teensyBreakout V2, debouncer
Parts:
- added 3V3: TERMINAL, Scott-Connectors:ED555/2DS
- added 5V: JST_PH_2.0_2P, Scott-Connectors:JST_PH_2.0_2P
- added ARD: JST_1.25_3P, Scott-Connectors:JST1.25_3P
- added BAT: JSTPH, Scott-Connectors:JST_PH_2.0_2P
- added C10, C7: 10µF, Scott-Electrical:0805
- added C11, C8: 1uF, Scott-Electrical:0603
- added C12: 0.1uF, Scott-Electrical:0603
- added C9: 10µF, Scott-Electrical:0603
- added CHG, PWR: (no value), Scott-Electrical:CHIPLED_0603
- added D2: MBR120, Scott-Electrical:SOD-123
- added J2, J3: 0, Scott-Electrical:0603
- added MCP: MCP73831, Scott-ICs:MICROBUILDER_SOT23-5
- added PRGM: JST_1.25_6P, Scott-Connectors:JST1.25_6P
- added Q2: DMG3415U, Scott-Electrical:SOT23-WIDE
- added R1, R6: (no value), Scott-Electrical:0603
- added R5: 1k, Scott-Electrical:0603
- added R7: 4.7k, Scott-Electrical:0603
- added R8: 10k, Scott-Electrical:0603
- added RA2: (no value), Scott-Electrical:RESCAF80P320X160X60-8N
- added REG: AP2112-3.3, Scott-ICs:MICROBUILDER_SOT23-5
- added RGB: LED_WS2812, Scott-ICs:LED-TRICOLOR-5050-IC
- added RST1: KMR2, Scott-Switches:BTN_KMR2_4.6X2.8
- added X1: ESP32_WROOM32, Scott-MCU:WROOM32
- J1: value TERMINAL -> (none); device Scott-Connectors:ED555/2DS -> Scott-Electrical:0603
- moved J1 46.4 mm to (55.6, 24.4)
- moved H2 32.7 mm to (40.1, 11.4)
- moved H1 29.5 mm to (5.84, -4.57)
Connections:
- new net A13_I35: RA2.4, RA2.6, X1.7
- new net EN: RA2.8, REG.3
- new net GPIO0: PRGM.1, X1.25
- new net IO13_A12: R6.2, X1.16
- new net N$1: PWR.C, R1.2
- new net N$10: R6.1, RGB.DIN
- new net N$5: CHG.C, R5.1
- new net N$6: MCP.1, R5.2
- new net N$8: MCP.5, R7.1
- new net N$9: C7.1, D2.C, J1.2, Q2.2, RA2.1, REG.1
- new net RESET: C11.1, PRGM.2, R8.1, RST1.B, RST1.B', X1.3
- new net RXARD: ARD.3, U$1.D0
- new net RXD0: J3.1, PRGM.4, X1.34
- new net RXESP: J2.2, U$1.D7
- new net TXARD: ARD.1, U$1.D1
- new net TXD0: J2.1, PRGM.3, X1.35
- new net TXESP: J3.2, U$1.D8
- new net VBAT: BAT.2, C10.1, MCP.3, Q2.3, RA2.3
- new net VBUS: 5V.2, CHG.A, D2.A, J1.1, MCP.4, Q2.1, RA2.2
- net 3.3V: now also 3V3.1, C12.1, C8.1, C9.1, PRGM.6, PWR.A, R8.2, REG.5, RGB.VDD, X1.2; no longer J1.1
- net GND: now also 3V3.2, 5V.1, ARD.2, BAT.1, C10.2, C11.2, C12.2, C7.2, C8.2, C9.2, MCP.2, PRGM.5, R1.1, R7.2, RA2.5, RA2.7, REG.2, RGB.VSS, RST1.A, RST1.A', X1.1, X1.15, X1.38, X1.P$1; no longer J1.2
Routing:
- net 3.3V: track 76.4 -> 154.0 mm, vias 2 -> 4
- net RXESP: track 0.00 -> 50.3 mm
- net RESET: track 0.00 -> 47.4 mm, vias 0 -> 2
- net VBUS: track 0.00 -> 46.4 mm
- net TXESP: track 0.00 -> 46.0 mm
- net VBAT: track 0.00 -> 31.1 mm, vias 0 -> 2
- net TXD0: track 0.00 -> 29.5 mm, vias 0 -> 4
- net RXD0: track 0.00 -> 29.3 mm, vias 0 -> 4
- net A13_I35: track 0.00 -> 15.7 mm
- net N$9: track 0.00 -> 10.4 mm
- net IO13_A12: track 0.00 -> 8.24 mm
- net GPIO0: track 0.00 -> 7.02 mm
- net N$6: track 0.00 -> 6.84 mm
- net GND: track 6.55 -> 0.00 mm, vias 13 -> 75
- net N$10: track 0.00 -> 4.08 mm
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Other:
- board size 29 x 47.2 mm -> 69.5 x 48.8 mm
- board text added: "3V3 Reg/Filter"
- board text added: "LiPo Charging"
- board text added: "Teensy Adapter V2 Feb 23, 2020"
- board text removed: "Teensy Adapter V1 Jan 16, 2020"

Commit message: bump pcb 2/24
Parts:
- IOEXP_1, IOEXP_2: value JST_1.25_6P -> JST_1.25_7P; device Scott-Connectors:JST1.25_6P -> Scott-Connectors:JST1.25_7P
- moved TB_PWM 1.78 mm to (31.8, 5.84)
- moved IOEXP_1 0.89 mm to (31.8, 20.7)
Connections:
- new net RST1: IOEXP_1.7, U$1.D9
- new net RST2: IOEXP_2.7, U$1.D10
Routing:
- net RST2: track 0.00 -> 32.9 mm, vias 0 -> 1
- net RST1: track 0.00 -> 21.1 mm
- net RXESP: track 50.3 -> 53.8 mm
- net TXESP: track 46.0 -> 49.4 mm
- net SDA: track 38.6 -> 40.7 mm
- net 3.3V: track 154.0 -> 155.4 mm
- net SCL: track 40.7 -> 41.5 mm
Other:
- board text added: "Teensy Adapter V2.1 Feb 24, 2020"
- board text removed: "Teensy Adapter V2 Feb 23, 2020"
