File: Electrical/PCB/TeensyBreakout/TeensyBreakout.sch (EAGLE design)
At the start: 7 parts, among them J1 TERMINAL

Commit message: teensyBreakout V2, debouncer
Parts:
- added 3V3: TERMINAL, Scott-Connectors:TERMINAL
- added 5V: JST_PH_2.0_2P, Scott-Connectors:JST_PH_2.0_2P
- added ARD: JST_1.25_3P, Scott-Connectors:JST_1.25_3P
- added BAT: JSTPH, Scott-Connectors:JST_PH_2.0_2P
- added C10, C7: 10µF, Scott-Electrical:CAP_CERAMIC_0805
- added C11, C8: 1uF, Scott-Electrical:CAP_CERAMIC_0603
- added C12: 0.1uF, Scott-Electrical:CAP_CERAMIC_0603
- added C9: 10µF, Scott-Electrical:CAP_CERAMIC_0603
- added CHG, PWR: (no value), Scott-Electrical:LED0603
- added D2: MBR120, Scott-Electrical:DIODE-SCHOTTKYSOD-123
- added J2, J3: 0, Scott-Electrical:RESISTOR0603
- added MCP: MCP73831, Scott-ICs:MCP73831/2
- added PRGM: JST_1.25_6P, Scott-Connectors:JST_1.25_6P
- added Q2: DMG3415U, Scott-Electrical:MOSFET-PWIDE
- added R1, R6: (no value), Scott-Electrical:RESISTOR0603
- added R5: 1k, Scott-Electrical:RESISTOR0603
- added R7: 4.7k, Scott-Electrical:RESISTOR0603
- added R8: 10k, Scott-Electrical:RESISTOR0603
- added RA2: (no value), Scott-Electrical:RESISTOR_ARRAY_1206_SEPARATE_REVERSE
- added REG: AP2112-3.3, Scott-ICs:VREG_SOT23-5
- added RGB: LED_WS2812, Scott-ICs:LED_WS2812
- added RST1: KMR2, Scott-Switches:SWITCH_TACT_SMT4.6X2.8
- added X1: ESP32_WROOM32, Scott-MCU:ESP32_WROOM32
- J1: value TERMINAL -> (none); device Scott-Connectors:TERMINAL -> Scott-Electrical:RESISTOR0603
Connections:
- new net A13_I35: RA2@3.1, RA2@4.2, X1.I35/A1_7
- new net EN: RA2@1.1, REG.EN
- new net GPIO0: PRGM.1, X1.IO0/A2_1
- new net IO13_A12: R6.2, X1.IO13/A2_4
- new net N$1: PWR.C, R1.2
- new net N$10: R6.1, RGB.DI
- new net N$5: CHG.C, R5.1
- new net N$6: MCP.STAT, R5.2
- new net N$8: MCP.PROG, R7.1
- new net N$9: C7.1, D2.C, J1.2, Q2.S, RA2@1.2, REG.IN
- new net RESET: C11.1, PRGM.2, R8.1, RST1.S, RST1.S1, X1.EN
- new net RXARD: ARD.3, U$1.D0
- new net RXD0: J3.1, PRGM.4, X1.RXD0
- new net RXESP: J2.2, U$1.D7
- new net TXARD: ARD.1, U$1.D1
- new net TXD0: J2.1, PRGM.3, X1.TXD0
- new net TXESP: J3.2, U$1.D8
- new net VBAT: BAT.2, C10.1, MCP.VBAT, Q2.D, RA2@3.2
- new net VBUS: 5V.2, CHG.A, D2.A, J1.1, MCP.VDD, Q2.G, RA2@2.2
- net 3.3V: now also 3V3.1, C12.1, C8.1, C9.1, PRGM.6, PWR.A, R8.2, REG.OUT, RGB.VDD, X1.3.3V; no longer J1.1
- net GND: now also 3V3.2, 5V.1, ARD.2, BAT.1, C10.2, C11.2, C12.2, C7.2, C8.2, C9.2, MCP.VSS, PRGM.5, R1.1, R7.2, RA2@2.1, RA2@4.1, REG.GND, RGB.VSS, RST1.P, RST1.P1, X1.GND; no longer J1.2
Other:
- note added: "1.0K = 1000mA"
- note added: "10K = 100mA"
- note added: "2.0K = 500mA"
- note added: "5.0K = 200mA"
- note added: "LED"
- note added: "LIPO CHARGING"
- note added: "MCU"
- note added: "POWER AND FILTERING"
- note added: "RESET"
- note added: "Strap Pin: IO0,IO2,IO5,IO12,IO15 -- Do not use Can only use for I2C: IO16,IO17 VBAT SENSE: IO35 RGBLED: IO13"

Commit message: bump pcb 2/24
Parts:
- IOEXP_1, IOEXP_2: value JST_1.25_6P -> JST_1.25_7P; device Scott-Connectors:JST_1.25_6P -> Scott-Connectors:JST_1.25_7P
Connections:
- new net RST1: IOEXP_1.7, U$1.D9
- new net RST2: IOEXP_2.7, U$1.D10
Changed lines of the file:
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@@
 <setting verticaltext="up"/>
 </settings>
-<grid distance="0.05" unitdist="inch" unit="inch" style="lines" multiple="1" display="no" altdistance="0.01" altunitdist="inch" altunit="inch"/>
+<grid distance="0.1" unitdist="inch" unit="inch" style="lines" multiple="1" display="no" altdistance="0.01" altunitdist="inch" altunit="inch"/>
 <layers>
 <layer number="1" name="Top" color="4" fill="1" visible="no" active="no"/>
@@
 <parts>
 <part name="U$1" library="Scott-MCU" deviceset="TEENSY4.0" device=""/>
-<part name="IOEXP_1" library="Scott-Connectors" deviceset="JST_1.25_6P" device=""/>
-<part name="IOEXP_2" library="Scott-Connectors" deviceset="JST_1.25_6P" device=""/>
+<part name="IOEXP_1" library="Scott-Connectors" deviceset="JST_1.25_7P" device=""/>
+<part name="IOEXP_2" library="Scott-Connectors" deviceset="JST_1.25_7P" device=""/>
 <part name="U$2" library="Scott-Electrical" deviceset="SUPPLY_3.3V" device=""/>
 <part name="GND1" library="Scott-Electrical" deviceset="SUPPLY_GND" device=""/>
@@
 <instances>
 <instance part="U$1" gate="G$1" x="-2.54" y="0" smashed="yes"/>
-<instance part="IOEXP_1" gate="&gt;NAME" x="-49.53" y="39.37" smashed="yes">
-<attribute name="NAME" x="-49.53" y="36.83" size="1.778" layer="95" font="vector" align="top-center"/>
-</instance>
-<instance part="IOEXP_2" gate="&gt;NAME" x="-26.67" y="39.37" smashed="yes">
-<attribute name="NAME" x="-26.67" y="36.83" size="1.778" layer="95" font="vector" align="top-center"/>
-</instance>
-<instance part="U$2" gate="G$1" x="-58.42" y="52.07" smashed="yes" rot="R90"/>
-<instance part="GND1" gate="1" x="-53.34" y="55.88" smashed="yes" rot="R180"/>
+<instance part="IOEXP_1" gate="&gt;NAME" x="-58.42" y="39.37" smashed="yes">
+<attribute name="NAME" x="-58.42" y="36.83" size="1.778" layer="95" font="vector" align="top-center"/>
+</instance>
+<instance part="IOEXP_2" gate="&gt;NAME" x="-25.4" y="39.116" smashed="yes">
+<attribute name="NAME" x="-25.4" y="36.576" size="1.778" layer="95" font="vector" align="top-center"/>
+</instance>
+<instance part="U$2" gate="G$1" x="-68.58" y="52.07" smashed="yes" rot="R90"/>
+<instance part="GND1" gate="1" x="-63.5" y="55.88" smashed="yes" rot="R180"/>
 <instance part="U$3" gate="G$1" x="-3.81" y="71.12" smashed="yes" rot="R90"/>
 <instance part="GND2" gate="1" x="-3.81" y="78.74" smashed="yes" rot="R270"/>
@@
 <segment>
 <pinref part="IOEXP_1" gate="&gt;NAME" pin="2"/>
-<wire x1="-53.34" y1="49.53" x2="-53.34" y2="53.34" width="0.1524" layer="91"/>
+<wire x1="-63.5" y1="49.53" x2="-63.5" y2="53.34" width="0.1524" layer="91"/>
 <pinref part="IOEXP_2" gate="&gt;NAME" pin="2"/>
-<wire x1="-53.34" y1="53.34" x2="-30.48" y2="53.34" width="0.1524" layer="91"/>
-<wire x1="-30.48" y1="53.34" x2="-30.48" y2="49.53" width="0.1524" layer="91"/>
+<wire x1="-63.5" y1="53.34" x2="-30.48" y2="53.34" width="0.1524" layer="91"/>
+<wire x1="-30.48" y1="53.34" x2="-30.48" y2="49.276" width="0.1524" layer="91"/>
 <pinref part="GND1" gate="1" pin="GND"/>
-<junction x="-53.34" y="53.34"/>
+<junction x="-63.5" y="53.34"/>
 </segment>
 <segment>
@@
 <segment>
 <pinref part="IOEXP_1" gate="&gt;NAME" pin="3"/>
-<wire x1="-50.8" y1="49.53" x2="-50.8" y2="54.61" width="0.1524" layer="91"/>
-<wire x1="-50.8" y1="54.61" x2="-27.94" y2="54.61" width="0.1524" layer="91"/>
+<wire x1="-60.96" y1="49.53" x2="-60.96" y2="54.61" width="0.1524" layer="91"/>
+<wire x1="-60.96" y1="54.61" x2="-27.94" y2="54.61" width="0.1524" layer="91"/>
 <pinref part="IOEXP_2" gate="&gt;NAME" pin="3"/>
-<wire x1="-27.94" y1="54.61" x2="-27.94" y2="49.53" width="0.1524" layer="91"/>
+<wire x1="-27.94" y1="54.61" x2="-27.94" y2="49.276" width="0.1524" layer="91"/>
 <label x="-27.94" y="49.53" size="1.778" layer="95" rot="R90"/>
 </segment>
@@
 <segment>
 <pinref part="IOEXP_1" gate="&gt;NAME" pin="4"/>
-<wire x1="-48.26" y1="49.53" x2="-48.26" y2="55.88" width="0.1524" layer="91"/>
+<wire x1="-58.42" y1="49.53" x2="-58.42" y2="55.88" width="0.1524" layer="91"/>
 <pinref part="IOEXP_2" gate="&gt;NAME" pin="4"/>
-<wire x1="-48.26" y1="55.88" x2="-25.4" y2="55.88" width="0.1524" layer="91"/>
-<wire x1="-25.4" y1="55.88" x2="-25.4" y2="49.53" width="0.1524" layer="91"/>
+<wire x1="-58.42" y1="55.88" x2="-25.4" y2="55.88" width="0.1524" layer="91"/>
+<wire x1="-25.4" y1="55.88" x2="-25.4" y2="49.276" width="0.1524" layer="91"/>
 <label x="-25.4" y="50.8" size="1.778" layer="95" rot="R90"/>
 </segment>
@@
 <segment>
 <pinref part="IOEXP_1" gate="&gt;NAME" pin="5"/>
-<wire x1="-45.72" y1="49.53" x2="-45.72" y2="60.96" width="0.1524" layer="91"/>
-<label x="-45.72" y="55.88" size="1.778" layer="95" rot="R90"/>
+<wire x1="-55.88" y1="49.53" x2="-55.88" y2="60.96" width="0.1524" layer="91"/>
+<label x="-55.88" y="55.88" size="1.778" layer="95" rot="R90"/>
 </segment>
 <segment>
@@
 <segment>
 <pinref part="IOEXP_1" gate="&gt;NAME" pin="6"/>
-<wire x1="-43.18" y1="49.53" x2="-43.18" y2="60.96" width="0.1524" layer="91"/>
-<label x="-43.18" y="55.88" size="1.778" layer="95" rot="R90"/>
+<wire x1="-53.34" y1="49.53" x2="-53.34" y2="60.96" width="0.1524" layer="91"/>
+<label x="-53.34" y="55.88" size="1.778" layer="95" rot="R90"/>
 </segment>
 <segment>
@@
 <segment>
 <pinref part="IOEXP_2" gate="&gt;NAME" pin="5"/>
-<wire x1="-22.86" y1="49.53" x2="-22.86" y2="60.96" width="0.1524" layer="91"/>
+<wire x1="-22.86" y1="49.276" x2="-22.86" y2="60.96" width="0.1524" layer="91"/>
 <label x="-22.86" y="55.88" size="1.778" layer="95" rot="R90"/>
 </segment>
@@
 <segment>
 <pinref part="IOEXP_2" gate="&gt;NAME" pin="6"/>
-<wire x1="-20.32" y1="49.53" x2="-20.32" y2="60.96" width="0.1524" layer="91"/>
+<wire x1="-20.32" y1="49.276" x2="-20.32" y2="60.96" width="0.1524" layer="91"/>
 <label x="-20.32" y="55.88" size="1.778" layer="95" rot="R90"/>
 </segment>
@@
 <segment>
 <pinref part="IOEXP_1" gate="&gt;NAME" pin="1"/>
-<wire x1="-55.88" y1="49.53" x2="-55.88" y2="52.07" width="0.1524" layer="91"/>
-<wire x1="-55.88" y1="52.07" x2="-33.02" y2="52.07" width="0.1524" layer="91"/>
+<wire x1="-66.04" y1="49.53" x2="-66.04" y2="52.07" width="0.1524" layer="91"/>
+<wire x1="-66.04" y1="52.07" x2="-33.02" y2="52.07" width="0.1524" layer="91"/>
 <pinref part="IOEXP_2" gate="&gt;NAME" pin="1"/>
-<wire x1="-33.02" y1="52.07" x2="-33.02" y2="49.53" width="0.1524" layer="91"/>
+<wire x1="-33.02" y1="52.07" x2="-33.02" y2="49.276" width="0.1524" layer="91"/>
 <pinref part="U$2" gate="G$1" pin="3.3V"/>
-<junction x="-55.88" y="52.07"/>
+<junction x="-66.04" y="52.07"/>
 </segment>
 <segment>
@@
 </segment>
 </net>
+<net name="RST1" class="0">
+<segment>
+<pinref part="IOEXP_1" gate="&gt;NAME" pin="7"/>
+<wire x1="-50.8" y1="49.53" x2="-50.8" y2="60.96" width="0.1524" layer="91"/>
+<label x="-50.8" y="55.88" size="1.778" layer="95" rot="R90"/>
+</segment>
+<segment>
+<pinref part="U$1" gate="G$1" pin="D9"/>
+<wire x1="7.62" y1="22.86" x2="-5.08" y2="22.86" width="0.1524" layer="91"/>
+<label x="-5.08" y="22.86" size="1.778" layer="95"/>
+</segment>
+</net>
+<net name="RST2" class="0">
+<segment>
+<pinref part="IOEXP_2" gate="&gt;NAME" pin="7"/>
+<wire x1="-17.78" y1="49.276" x2="-17.78" y2="60.96" width="0.1524" layer="91"/>
+<label x="-17.78" y="55.88" size="1.778" layer="95" rot="R90"/>
+</segment>
+<segment>
+<pinref part="U$1" gate="G$1" pin="D10"/>
+<wire x1="7.62" y1="19.05" x2="-5.08" y2="19.05" width="0.1524" layer="91"/>
+<label x="-5.08" y="19.05" size="1.778" layer="95"/>
+</segment>
+</net>
